Commit message: Dodana ovira v collision_objects Obarval vacuum ON/OFF logs Barve v collision_objects Dodal dejanski prižig vakuuma v pick_and_place V hello_moveit_targets dodal spremenljivke za hitre in počasne gibe, nekaj kode tudi v pick_and_place Bolj točni collision_objects

File: src/fanuc_description/fanuc_m20ia_description/urdf/m20ia_urdf_macro.xacro (robot description, xacro)
@@ -41,5 +41,5 @@
     <link name="${prefix}base_link">
       <visual>
-        <origin xyz="0 0 0" rpy="0 0 0" />
+        <origin xyz="0 0 9.5" rpy="0 0 0" />
         <geometry>
           <mesh
@@ -325,5 +325,5 @@
     <link name="${prefix}wbase" />
     <joint name="${prefix}base_link-wbase" type="fixed">
-      <origin xyz=" 0  0  .425" rpy="0 0 0" />
+      <origin xyz=" 0  0  9.425" rpy="0 0 0" />
       <parent link="${prefix}base_link" />
       <child link="${prefix}wbase" />

File: src/fanuc_m20ia_moveit_config/config/fanuc_m20ia.urdf.xacro (robot description, xacro)
@@ -7,4 +7,10 @@
     <xacro:include filename="fanuc_m20ia.ros2_control.xacro" />
     <xacro:fanuc_m20ia_ros2_control name="FakeSystem" initial_positions_file="$(arg initial_positions_file)"/>
+    <link name="world"/>
+    <joint name="world_to_base_link" type="fixed">
+      <parent link="world"/>
+      <child link="base_link"/>
+      <origin xyz="0 0 0.095" rpy="0 0 0"/>
+    </joint>
     <link name="tool_link">
       <visual>
