Commit message: v pick_and_place dodana koda z aizvedbo več planov in execute najkrajšega joint zamiki v m20ia.urdf popravljeni m20ia_urdf_macro.xacro, sedaj generira enak urdf m20ia.urdf codex dodal varovalko v pick_and_place...

File: src/fanuc_description/fanuc_m20ia_description/urdf/m20ia.urdf (robot description, URDF)
Before this commit: robot fanuc_m20ia, 10 links, 9 joints
Joints:
- joint joint_4: origin xyz=0 0 0.250 rpy=0 0 0 -> xyz=0 0 0.150 rpy=0 0 0
- joint joint_5: origin xyz=0.835 0 0 rpy=0 0 0 -> xyz=0.860 0 0 rpy=0 0 0

File: src/fanuc_description/fanuc_m20ia_description/urdf/m20ia_urdf_macro.xacro (robot description, xacro)
@@ -5,5 +5,5 @@
 SPDX-License-Identifier: Apache-2.0
 -->
-<!-- URDF for M-20/25-18D (M-20iD/25) -->
+<!-- URDF macro matching urdf/m20ia.urdf for FANUC M-20iA -->
 <robot xmlns:xacro="http://wiki.ros.org/xacro">
   <xacro:macro
@@ -14,332 +14,271 @@
             child"
   >
-    <xacro:property name="j1_lower_limit" value="${radians(-185)}" />
-    <xacro:property name="j2_lower_limit" value="${radians(-100)}" />
-    <xacro:property name="j3_lower_limit" value="${radians(-90)}" />
-    <xacro:property name="j4_lower_limit" value="${radians(-200)}" />
-    <xacro:property name="j5_lower_limit" value="${radians(-179.999)}" />
-    <xacro:property name="j6_lower_limit" value="${radians(-450)}" />
-    <xacro:property name="j1_upper_limit" value="${radians(185)}" />
-    <xacro:property name="j2_upper_limit" value="${radians(160)}" />
-    <xacro:property name="j3_upper_limit" value="${radians(220)}" />
-    <xacro:property name="j4_upper_limit" value="${radians(200)}" />
-    <xacro:property name="j5_upper_limit" value="${radians(179.999)}" />
-    <xacro:property name="j6_upper_limit" value="${radians(450)}" />
-    <xacro:property name="j1_effort_limit" value="7000" />
-    <xacro:property name="j2_effort_limit" value="8000" />
-    <xacro:property name="j3_effort_limit" value="4000" />
-    <xacro:property name="j4_effort_limit" value="300" />
-    <xacro:property name="j5_effort_limit" value="300" />
-    <xacro:property name="j6_effort_limit" value="200" />
-    <xacro:property name="j1_velocity_limit" value="${radians(210)}" />
-    <xacro:property name="j2_velocity_limit" value="${radians(210)}" />
-    <xacro:property name="j3_velocity_limit" value="${radians(265)}" />
-    <xacro:property name="j4_velocity_limit" value="${radians(420)}" />
-    <xacro:property name="j5_velocity_limit" value="${radians(420)}" />
-    <xacro:property name="j6_velocity_limit" value="${radians(720)}" />
-    <!-- links -->
+    <!-- links: main serial chain -->
     <link name="${prefix}base_link">
       <visual>
-        <origin xyz="0 0 9.5" rpy="0 0 0" />
-        <geometry>
-          <mesh
-            filename="package://fanuc_m20ia_description/meshes/m20ia/visual/base_link.stl"
-          />
-        </geometry>
-      </visual>
-      <collision>
-        <origin xyz="0 0 0" rpy="0 0 0" />
-        <geometry>
-          <mesh
-            filename="package://fanuc_m20ia_description/meshes/m20ia/collision/base_link.stl"
-          />
-        </geometry>
-      </collision>
-      <inertial>
-        <mass value=" 45.8" />
-        <origin xyz="-.0767  .00288  .109" />
-        <inertia
-          ixx=" .497"
-          ixy=" .029"
-          ixz=" .0137"
-          iyy=" 1.1"
-          iyz=" .0000537"
-          izz=" 1.16"
-        />
-      </inertial>
-    </link>
-    <link name="${prefix}J1_link">
-      <visual>
-        <origin xyz="0 0 0" rpy="0 0 0" />
-        <geometry>
-          <mesh
-            filename="package://fanuc_m20ia_description/meshes/m20ia/visual/link_1.stl"
-          />
-        </geometry>
-      </visual>
-      <collision>
-        <origin xyz="0 0 0" rpy="0 0 0" />
-        <geometry>
-          <mesh
-            filename="package://fanuc_m20ia_description/meshes/m20ia/collision/link_1.stl"
-          />
-        </geometry>
-      </collision>
-      <inertial>
-        <mass value=" 62.8" />
-        <origin xyz=" .0158 -.0106 -.0831" />
-        <inertia
-          ixx=" 1.35"
-          ixy=" .133"
-          ixz="-.0417"
-          iyy=" 1.11"
-          iyz="-.108"
-          izz=" 1.3"
-        />
-      </inertial>
-    </link>
-    <link name="${prefix}J2_link">
-      <visual>
-        <origin xyz="0 0 0" rpy="0 0 0" />
-        <geometry>
-          <mesh
-            filename="package://fanuc_m20ia_description/meshes/m20ia/visual/link_2.stl"
-          />
-        </geometry>
-      </visual>
-      <collision>
-        <origin xyz="0 0 0" rpy="0 0 0" />
-        <geometry>
-          <mesh
-            filename="package://fanuc_m20ia_description/meshes/m20ia/collision/link_2.stl"
-          />
-        </geometry>
-      </collision>
-      <inertial>
-        <mass value=" 65.8" />
-        <origin xyz="-.0343 -.172  .38" />
-        <inertia
-          ixx=" 4.86"
-          ixy="-.0809"
-          ixz=" .0453"
-          iyy=" 4.98"
-          iyz="-.118"
-          izz=" .536"
-        />
-      </inertial>
-    </link>
-    <link name="${prefix}J3_link">
-      <visual>
-        <origin xyz="0 0 0" rpy="0 0 0" />
-        <geometry>
-          <mesh
-            filename="package://fanuc_m20ia_description/meshes/m20ia/visual/link_3.stl"
-          />
-        </geometry>
-      </visual>
-      <collision>
-        <origin xyz="0 0 0" rpy="0 0 0" />
-        <geometry>
-          <mesh
-            filename="package://fanuc_m20ia_description/meshes/m20ia/collision/link_3.stl"
-          />
-        </geometry>
-      </collision>
-      <inertial>
-        <mass value=" 52.9" />
-        <origin xyz=" .134  .00796  .103" />
-        <inertia
-          ixx=" .901"
-          ixy="-.0784"
-          ixz="-.294"
-          iyy=" 1.13"
-          iyz="-.0385"
-          izz=" 1.06"
-        />
-      </inertial>
-    </link>
-    <link name="${prefix}J4_link">
-      <visual>
-        <origin xyz="0 0 0" rpy="0 0 0" />
-        <geometry>
-          <mesh
-            filename="package://fanuc_m20ia_description/meshes/m20ia/visual/link_4.stl"
-          />
-        </geometry>
-      </visual>
-      <collision>
-        <origin xyz="0 0 0" rpy="0 0 0" />
-        <geometry>
-          <mesh
-            filename="package://fanuc_m20ia_description/meshes/m20ia/collision/link_4.stl"
-          />
-        </geometry>
-      </collision>
-      <inertial>
-        <mass value=" 20.2" />
-        <origin xyz=" .586 -.0481 -.000358" />
-        <inertia
-          ixx=" .0769"
-          ixy=" .053"
-          ixz="-.00106"
-          iyy=" .647"
-          iyz="-.0000313"
-          izz=" .656"
-        />
-      </inertial>
-    </link>
-    <link name="${prefix}J5_link">
-      <visual>
-        <origin xyz="0 0 0" rpy="0 0 0" />
-        <geometry>
-          <mesh
-            filename="package://fanuc_m20ia_description/meshes/m20ia/visual/link_5.stl"
-          />
-        </geometry>
-      </visual>
-      <collision>
-        <origin xyz="0 0 0" rpy="0 0 0" />
-        <geometry>
-          <mesh
-            filename="package://fanuc_m20ia_description/meshes/m20ia/collision/link_5.stl"
-          />
-        </geometry>
-      </collision>
-      <inertial>
-        <mass value=" 1.98" />
-        <origin xyz=" .0276 -.0121  .000000522" />
-        <inertia
-          ixx=" .00394"
-          ixy="-.000785"
-          ixz=" .0000000339"
-          iyy=" .00462"
-          iyz=" .00000000332"
-          izz=" .0041"
-        />
-      </inertial>
-    </link>
-    <link name="${prefix}J6_link">
-      <visual>
-        <origin xyz="0 0 0" rpy="0 0 0" />
-        <geometry>
-          <mesh
-            filename="package://fanuc_m20ia_description/meshes/m20ia/visual/link_6.stl"
-          />
-        </geometry>
-      </visual>
-      <collision>
-        <origin xyz="0 0 0" rpy="0 0 0" />
-        <geometry>
-          <mesh
-            filename="package://fanuc_m20ia_description/meshes/m20ia/collision/link_6.stl"
-          />
-        </geometry>
-      </collision>
-      <inertial>
-        <mass value=" .558" />
-        <origin xyz=" .0581 -.000000509  .000000147" />
-        <inertia
-          ixx=" .000585"
-          ixy="-.00000000703"
-          ixz=" .0000000019"
-          iyy=" .000433"
-          iyz=" .0000000227"
-          izz=" .000433"
-        />
-      </inertial>
-    </link>
-    <!-- joints -->
-    <joint name="${prefix}J1" type="revolute">
-      <origin xyz=" 0  0  .425" rpy="0 0 0" />
+        <origin rpy="0 0 0" xyz="0 0 0" />
+        <geometry>
+          <mesh filename="package://fanuc_m20ia_description/meshes/m20ia/visual/base_link.stl" />
+        </geometry>
+        <material name="">
+          <color rgba="0.2784313725490196 0.2784313725490196 0.2784313725490196 1.0" />
+        </material>
+      </visual>
+      <collision>
+        <origin rpy="0 0 0" xyz="0 0 0" />
+        <geometry>
+          <mesh filename="package://fanuc_m20ia_description/meshes/m20ia/collision/base_link.stl" />
+        </geometry>
+      </collision>
+      <inertial>
+        <mass value=" 32.5" />
+        <origin xyz="-.0269 -.0000215  .157" />
+        <inertia
+          ixx=" .556"
+          ixy="-.00546"
+          ixz="-.00524"
+          iyy=" .681"
+          iyz="-.000569"
+          izz=" .667"
+        />
+      </inertial>
+    </link>
+    <link name="${prefix}link_1">
+      <visual>
+        <origin rpy="0 0 0" xyz="0 0 0" />
+        <geometry>
+          <mesh filename="package://fanuc_m20ia_description/meshes/m20ia/visual/link_1.stl" />
+        </geometry>
+        <material name="">
+          <color rgba="0.96 0.76 0.13 1.0" />
+        </material>
+      </visual>
+      <collision>
+        <origin rpy="0 0 0" xyz="0 0 0" />
+        <geometry>
+          <mesh filename="package://fanuc_m20ia_description/meshes/m20ia/collision/link_1.stl" />
+        </geometry>
+      </collision>
+      <inertial>
+        <mass value=" 52.3" />
+        <origin xyz=" .0372  .00108 -.101" />
+        <inertia
+          ixx=" 1.85"
+          ixy="-.00339"
+          ixz="-.149"
+          iyy=" 1.15"
+          iyz="-.00387"
+          izz=" 1.52"
+        />
+      </inertial>
+    </link>
+    <link name="${prefix}link_2">
+      <visual>
+        <origin rpy="0 0 0" xyz="0 0 0" />
+        <geometry>
+          <mesh filename="package://fanuc_m20ia_description/meshes/m20ia/visual/link_2.stl" />
+        </geometry>
+        <material name="">
+          <color rgba="0.96 0.76 0.13 1.0" />
+        </material>
+      </visual>
+      <collision>
+        <origin rpy="0 0 0" xyz="0 0 0" />
+        <geometry>
+          <mesh filename="package://fanuc_m20ia_description/meshes/m20ia/collision/link_2.stl" />
+        </geometry>
+      </collision>
+      <inertial>
+        <mass value=" 92.7" />
+        <origin xyz="-.0012 -.000625  .461" />
+        <inertia
+          ixx=" 10.7"
+          ixy="-.00108"
+          ixz=" .00167"
+          iyy=" 10"
+          iyz=" .00496"
+          izz=" 1.7"
+        />
+      </inertial>
+    </link>
+    <link name="${prefix}link_3">
+      <visual>
+        <origin rpy="0 0 0" xyz="0 0 0" />
+        <geometry>
+          <mesh filename="package://fanuc_m20ia_description/meshes/m20ia/visual/link_3.stl" />
+        </geometry>
+        <material name="">
+          <color rgba="0.96 0.76 0.13 1.0" />
+        </material>
+      </visual>
+      <collision>
+        <origin rpy="0 0 0" xyz="0 0 0" />
+        <geometry>
+          <mesh filename="package://fanuc_m20ia_description/meshes/m20ia/collision/link_3.stl" />
+        </geometry>
+      </collision>
+      <inertial>
+        <mass value=" 17.2" />
+        <origin xyz=" .0221 -.00161  .0386" />
+        <inertia
+          ixx=" .21"
+          ixy="-.00523"
+          ixz="-.0224"
+          iyy=" .233"
+          iyz="-.00207"
+          izz=" .205"
+        />
+      </inertial>
+    </link>
+    <link name="${prefix}link_4">
+      <visual>
+        <origin rpy="0 0 0" xyz="0 0 0" />
+        <geometry>
+          <mesh filename="package://fanuc_m20ia_description/meshes/m20ia/visual/link_4.stl" />
+        </geometry>
+        <material name="">
+          <color rgba="0.96 0.76 0.13 1.0" />
+        </material>
+      </visual>
+      <collision>
+        <origin rpy="0 0 0" xyz="0 0 0" />
+        <geometry>
+          <mesh filename="package://fanuc_m20ia_description/meshes/m20ia/collision/link_4.stl" />
+        </geometry>
+      </collision>
+      <inertial>
+        <mass value=" 14.2" />
+        <origin xyz=" .524  .00617 -.0000045" />
+        <inertia
+          ixx=" .0578"
+          ixy=" .00266"
+          ixz="-.00000254"
+          iyy=" .638"
+          iyz=" .00000567"
+          izz=" .654"
+        />
+      </inertial>
+    </link>
+    <link name="${prefix}link_5">
+      <visual>
+        <origin rpy="0 0 0" xyz="0 0 0" />
+        <geometry>
+          <mesh filename="package://fanuc_m20ia_description/meshes/m20ia/visual/link_5.stl" />
+        </geometry>
+        <material name="">
+          <color rgba="0.96 0.76 0.13 1.0" />
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
File: src/fanuc_m20ia_moveit_config/config/fanuc_m20ia.urdf.xacro (robot description, xacro)
@@ -7,10 +7,4 @@
     <xacro:include filename="fanuc_m20ia.ros2_control.xacro" />
     <xacro:fanuc_m20ia_ros2_control name="FakeSystem" initial_positions_file="$(arg initial_positions_file)"/>
-    <link name="world"/>
-    <joint name="world_to_base_link" type="fixed">
-      <parent link="world"/>
-      <child link="base_link"/>
-      <origin xyz="0 0 0.095" rpy="0 0 0"/>
-    </joint>
     <link name="tool_link">
       <visual>
